Commit message: fixed laser ray missing and rviz crash issue with fixed link as odom

File: src/myhamster/myhamster_simulation/urdf/front_wheel.urdf.xacro (robot description, xacro)
@@ -15,5 +15,5 @@
         <origin xyz="0 0 0" rpy="1.57 0 0" />
         <geometry>
-          <mesh filename="package://hamster_vehicle_description/meshes/hamster_wheel.dae" />
+          <mesh filename="package://myhamster_simulation/meshes/hamster_wheel.dae" />
         </geometry>
       </visual>

File: src/myhamster/myhamster_simulation/urdf/hamster.urdf.xacro (robot description, xacro)
@@ -1,6 +1,6 @@
 <?xml version="1.0"?>
 <robot name="hamster" xmlns:xacro="http://www.ros.org/wiki/xacro">
-  <xacro:include filename="$(find hamster_vehicle_description)/urdf/front_wheel.urdf.xacro" />
-  <xacro:include filename="$(find hamster_vehicle_description)/urdf/rear_wheel.urdf.xacro" />
+  <xacro:include filename="$(find myhamster_simulation)/urdf/front_wheel.urdf.xacro" />
+  <xacro:include filename="$(find myhamster_simulation)/urdf/rear_wheel.urdf.xacro" />
   <xacro:macro name="solid_cuboid_inertia" params="w h d m">
   <inertia  ixx="${m*(h*h+d*d)/12}" ixy = "0" ixz = "0"
@@ -19,5 +19,5 @@
     <visual>
       <geometry>
-        <mesh filename="package://hamster_vehicle_description/meshes/shell.dae" />
+        <mesh filename="package://myhamster_simulation/meshes/shell.dae" />
       </geometry>
     </visual>
@@ -77,5 +77,5 @@
     <visual>
       <geometry>
-        <mesh filename="package://hamster_vehicle_description/meshes/A2_lidar.dae" />
+        <mesh filename="package://myhamster_simulation/meshes/A2_lidar.dae" />
       </geometry>
     </visual>
@@ -90,8 +90,8 @@
       <geometry>
         <xacro:if value="${version == 'V7'}">
-        <mesh filename="package://hamster_vehicle_description/meshes/d415.stl" />
+        <mesh filename="package://myhamster_simulation/meshes/d415.stl" />
         </xacro:if>
         <xacro:if value="${version == 'V6'}">
-        <mesh filename="package://hamster_vehicle_description/meshes/camera.stl" />
+        <mesh filename="package://myhamster_simulation/meshes/camera.stl" />
         </xacro:if>
       </geometry>
@@ -109,5 +109,5 @@
   <gazebo>
     <plugin name="gazebo_ros_control" filename="libgazebo_ros_control.so">
-      <robotNamespace>$(arg agent)</robotNamespace>
+      <robotNamespace></robotNamespace>
       <robotSimType>gazebo_ros_control/DefaultRobotHWSim</robotSimType>
       <legacyModeNS>true</legacyModeNS>
@@ -116,5 +116,5 @@
   <gazebo>
     <plugin name="gazebo_ackermann_drive" filename="libgazebo_ackermann_drive.so">
-      <robotNamespace>$(arg agent)</robotNamespace>
+      <robotNamespace></robotNamespace>
       <robotBaseLink>base_link</robotBaseLink>
       <wheelRadius>0.029</wheelRadius>
@@ -153,10 +153,10 @@
         <xyzOffset>0 0 0</xyzOffset>
         <rpyOffset>0 0 0</rpyOffset>
-        <frameName>$(arg agent)/imu_link</frameName>
+        <frameName>imu_link</frameName>
       </plugin>
     </sensor>
   </gazebo>
   <gazebo reference="lidar_link">
-    <sensor type="gpu_ray" name="head_hokuyo_sensor">
+    <sensor type="ray" name="head_hokuyo_sensor">
       <pose>0 0 0 0 0 0</pose>
       <visualize>false</visualize>
@@ -182,5 +182,5 @@
         </noise>
       </ray>
-      <plugin name="gazebo_ros_head_hokuyo_controller" filename="libgazebo_ros_gpu_laser.so">
+      <plugin name="gazebo_ros_head_hokuyo_controller" filename="libgazebo_ros_laser.so">
         <topicName>scan</topicName>
         <frameName>lidar_link</frameName>
@@ -262,5 +262,5 @@
           <imageTopicName>image_raw</imageTopicName>
           <cameraInfoTopicName>camera_info</cameraInfoTopicName>
-          <frameName>$(arg agent)/camera_link</frameName>
+          <frameName>camera_link</frameName>
           <hackBaseline>0.07</hackBaseline>
           <distortionK1>0.0</distortionK1>

File: src/myhamster/myhamster_simulation/urdf/rear_wheel.urdf.xacro (robot description, xacro)
@@ -15,5 +15,5 @@
         <origin xyz="0 0 0" rpy="1.57 0 0" />
         <geometry>
-          <mesh filename="package://hamster_vehicle_description/meshes/hamster_wheel.dae" />
+          <mesh filename="package://myhamster_simulation/meshes/hamster_wheel.dae" />
         </geometry>
       </visual>
